Commit message: combine openmanipulator-x to tb3

File: src/turtlebot3/turtlebot3/turtlebot3_description/urdf/turtlebot3_burger.urdf (robot description, URDF)
Before this commit: robot turtlebot3_burger, 7 links, 6 joints
Links:
- added link end_effector_link, mass 0.001; visual box size=0.01 0.01 0.01
- added link gripper_link, mass 0.017; collision mesh filename=package://open_manipulator_x_description/meshes/link_grip_l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 scale=0.001 0.001 0.001; visual mesh filename=package://open_manipulator_x_description/meshes/link_grip_l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 scale=0.001 0.001 0.001
- added link gripper_link_sub, mass 0.017; collision mesh filename=package://open_manipulator_x_description/meshes/link_grip_r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 scale=0.001 0.001 0.001; visual mesh filename=package://open_manipulator_x_description/meshes/link_grip_r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 scale=0.001 0.001 0.001
- added link link1, mass 7.9119962e-02; collision mesh filename=package://open_manipulator_x_description/meshes/link1.stl scale=0.001 0.001 0.001; visual mesh filename=package://open_manipulator_x_description/meshes/link1.stl scale=0.001 0.001 0.001
- added link link2, mass 9.8406837e-02; collision mesh filename=package://open_manipulator_x_description/meshes/link2.stl scale=0.001 0.001 0.001; visual mesh filename=package://open_manipulator_x_description/meshes/link2.stl scale=0.001 0.001 0.001
- added link link3, mass 1.3850917e-01; collision mesh filename=package://open_manipulator_x_description/meshes/link3.stl scale=0.001 0.001 0.001; visual mesh filename=package://open_manipulator_x_description/meshes/link3.stl scale=0.001 0.001 0.001
- added link link4, mass 1.3274562e-01; collision mesh filename=package://open_manipulator_x_description/meshes/link4.stl scale=0.001 0.001 0.001; visual mesh filename=package://open_manipulator_x_description/meshes/link4.stl scale=0.001 0.001 0.001
- added link link5, mass 1.4327573e-01; collision mesh filename=package://open_manipulator_x_description/meshes/link5.stl scale=0.001 0.001 0.001; visual mesh filename=package://open_manipulator_x_description/meshes/link5.stl scale=0.001 0.001 0.001
Joints:
- added joint end_effector_joint: type fixed, parent link5, child end_effector_link, origin xyz=0.126 0.0 0.0 rpy=0 0 0
- added joint gripper: type prismatic, parent link5, child gripper_link, origin xyz=0.0817 0.021 0.0 rpy=0 0 0, axis 0 1 0, limit lower=-0.010 upper=0.019 effort=1 velocity=4.8
- added joint gripper_sub: type prismatic, parent link5, child gripper_link_sub, origin xyz=0.0817 -0.021 0 rpy=0 0 0, axis 0 -1 0, limit lower=-0.010 upper=0.019 effort=1 velocity=4.8, mimic joint=gripper multiplier=1
- added joint joint1: type revolute, parent link1, child link2, origin xyz=0.012 0.0 0.017 rpy=0 0 0, axis 0 0 1, limit lower=-2.82743338823 upper=2.82743338823 effort=1 velocity=4.8
- added joint joint2: type revolute, parent link2, child link3, origin xyz=0.0 0.0 0.0595 rpy=0 0 0, axis 0 1 0, limit lower=-1.79070781255 upper=1.57079632679 effort=1 velocity=4.8
- added joint joint3: type revolute, parent link3, child link4, origin xyz=0.024 0 0.128 rpy=0 0 0, axis 0 1 0, limit lower=-0.94247779607 upper=1.38230076758 effort=1 velocity=4.8
- added joint joint4: type revolute, parent link4, child link5, origin xyz=0.124 0.0 0.0 rpy=0 0 0, axis 0 1 0, limit lower=-1.79070781255 upper=2.04203522483 effort=1 velocity=4.8
- added joint world_fixed: type fixed, parent base_link, child link1, origin xyz=0.06 0 0.01 rpy=0 0 0
